File: Hardware/PDB.kicad_sch (KiCad schematic)
At the start: 50 parts, among them J1 Conn_01x02, J2 Conn_01x02, J3 Conn_01x02, J4 Conn_01x02, J5 Conn_01x02, Q1 Q_PMOS_GDS, U1 TPS54302, U2 TPS54302, U3 AP2112K-1.8, U4 INA219AxD

Commit message: Even more small changes
Changed lines of the file:
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@@
 	(text "MOUNTING HOLES"
 		(exclude_from_sim no)
-		(at 36.322 159.004 0)
+		(at 35.306 159.004 0)
 		(effects
 			(font
@@
 	(text "INTERFACE"
 		(exclude_from_sim no)
-		(at 163.576 90.424 0)
+		(at 163.576 90.932 0)
 		(effects
 			(font
@@
 	(text "5V REGULATOR"
 		(exclude_from_sim no)
-		(at 32.258 91.44 0)
+		(at 32.258 90.932 0)
 		(effects
 			(font
@@
 	(text "1.8V REGULATOR"
 		(exclude_from_sim no)
-		(at 158.496 18.288 0)
+		(at 159.258 18.288 0)
 		(effects
 			(font
@@
 	(wire
 		(pts
-			(xy 171.45 124.46) (xy 171.45 125.73)
+			(xy 172.72 123.19) (xy 172.72 125.73)
 		)
 		(stroke
@@
 	(wire
 		(pts
-			(xy 171.45 125.73) (xy 165.1 125.73)
+			(xy 172.72 125.73) (xy 165.1 125.73)
 		)
 		(stroke
@@
 	(symbol
 		(lib_id "power:PWR_FLAG")
-		(at 171.45 124.46 0)
+		(at 172.72 123.19 0)
 		(mirror y)
 		(unit 1)
@@
 		(dnp no)
 		(property "Reference" "#FLG04"
-			(at 171.45 122.555 0)
+			(at 172.72 121.285 0)
 			(effects
 				(font
@@
 		)
 		(property "Value" "PWR_FLAG"
-			(at 171.45 120.65 0)
+			(at 172.72 119.38 0)
 			(effects
 				(font
@@
 		)
 		(property "Footprint" ""
-			(at 171.45 124.46 0)
+			(at 172.72 123.19 0)
 			(effects
 				(font
@@
 		)
 		(property "Datasheet" "~"
-			(at 171.45 124.46 0)
+			(at 172.72 123.19 0)
 			(effects
 				(font
@@
 		)
 		(property "Description" "Special symbol for telling ERC where power comes from"
-			(at 171.45 124.46 0)
+			(at 172.72 123.19 0)
 			(effects
 				(font

Commit message: More changes
Parts:
- removed L2, L4: 1uH, Inductor_SMD:L_1206_3216Metric, symbol Device:L_Ferrite
- added C18: 47uF, Capacitor_SMD:C_1206_3216Metric, symbol Device:C
- added C19: 10uF, Capacitor_SMD:C_1206_3216Metric, symbol Device:C
- added FB1, FB2: FerriteBead, Inductor_SMD:L_0805_2012Metric, symbol Device:FerriteBead
- C10: value 47uF -> 10uF
Connections:
- net +3.3V: now also FB1.2
- net +5V: now also C19.1, FB2.2; no longer C12.1
- net GND: now also C18.2, C19.2
- net at L3.2: now also C12.1, FB2.1
- net at L1.2: now also C18.1, FB1.1
Other:
- note added: "100ohms @ 100MHz"
- moved on the sheet: C12, C13, R3, R4

Commit message: More changes
Connections:
- net 5V_FER: now reaches C12.1, FB2.1, L3.2
- net 3V3_FER: now reaches C18.1, FB1.1, L1.2
Other:
- note added: "I2c Address: 0x4240"
- moved on the sheet: C1, C10, C11, C12, C13, C14, C15, C16, C17, C18, C19, C2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
